File: scsiemu.sch (KiCad schematic (older format))
At the start: 32 parts, among them J1 RasPi, J2 SCSI, J3 USB_POWER, J4 POWER 5V, J5 I2C, U1 74LS641-1, U2 74LS641-1, U3 74LS641-1, U4 74LS641-1

Commit message: Internal 50pin version (#1)
Parts:
- removed J2: SCSI, local_lib:DSUB50P, symbol local_lib:DSUB_SCSI
- removed J5: I2C, Connector_JST:JST_PH_S3B-PH-K_1x03_P2.00mm_Horizontal, symbol Connector:Conn_01x03_Male
- removed RN10, RN5, RN7, RN8: 220, Resistor_SMD:R_Cat16-8, symbol Device:R_Pack08
- removed RN11, RN6, RN9: 330, Resistor_SMD:R_Cat16-8, symbol Device:R_Pack08
- added C10, C11, C6, C8: 10u, Capacitor_SMD:C_1206_3216Metric_Pad1.42x1.75mm_HandSolder, symbol Device:C
- added C7, C9: 2.2u, Capacitor_SMD:C_0603_1608Metric_Pad1.05x0.95mm_HandSolder, symbol Device:C
- added D2: SBD, local_lib:D_SOD-123_HandSoldering, symbol Device:D_ALT
- added J2: SCSI, Connector_PinHeader_2.54mm:PinHeader_2x25_P2.54mm_Horizontal, symbol Connector_Generic:Conn_02x25_Odd_Even
- added J5: POWER 5V, Connector_JST:JST_XH_B2B-XH-A_1x02_P2.50mm_Vertical, symbol Connector:Conn_01x02_Male
- added J6: AT Power 5V (171826-4), local_lib:Molex_171826-4, symbol Connector_Generic:Conn_01x04
- added J7: I2C Ext, Connector_JST:JST_XH_B6B-XH-A_1x06_P2.50mm_Vertical, symbol Connector_Generic:Conn_01x06
- added J8: AT Power 5V (641737-1), local_lib:TE_641737-1, symbol Connector_Generic:Conn_01x04
- added LED2: LED ACT, LED_SMD:LED_0603_1608Metric_Pad1.05x0.95mm_HandSolder, symbol Device:LED
- added MH1, MH10, MH2, MH3, MH4, MH9: Raspi Mount, MountingHole:MountingHole_2.2mm_M2, symbol Connector_Generic:Conn_01x01
- added MH11, MH12, MH5, MH6, MH7, MH8: HDD Mount, MountingHole:MountingHole_3.5mm, symbol Connector_Generic:Conn_01x01
- added R2: 2.2k, Resistor_SMD:R_0603_1608Metric_Pad1.05x0.95mm_HandSolder, symbol Device:R
- added R3: 2.7k, Resistor_SMD:R_0603_1608Metric_Pad1.05x0.95mm_HandSolder, symbol Device:R
- added R4: 1k, Resistor_SMD:R_0603_1608Metric_Pad1.05x0.95mm_HandSolder, symbol Device:R
- added U5, U6: DS2105Z, Package_SO:SOIC-16_3.9x9.9mm_P1.27mm, symbol local_lib:DS2105Z
- added U7, U8: TL2218-285, Package_SO:TSSOP-20_4.4x6.5mm_P0.65mm, symbol local_lib:TL2218-285
- C1, C2, C4: value 0.1u JB -> 0.1u
- C3: value 0.1u JIS B -> 0.1u
- C5: value 10u JB -> 10u
- D1: footprint cd_device:D_SOD-123_HandSoldering -> local_lib:D_SOD-123_HandSoldering
- F1: value 1A -> 750mA ~~ 1A (0ZCJ0075FF2E)
- F2: value 1A -> 2A (0685T2000-01)
- J4: footprint Connector_JST:JST_PH_S2B-PH-K_1x02_P2.00mm_Horizontal -> Connector_JST:JST_XH_B2B-XH-A_1x02_P2.50mm_Vertical
- LED1: value LED ACT -> LED PWR; footprint LED_THT:LED_D3.0mm -> LED_SMD:LED_0603_1608Metric_Pad1.05x0.95mm_HandSolder
Connections:
- net labels added: 5V_DC, AT_5V_DC, AT_POWER_ON, EXT1, EXT2, S_ACK, S_ATN, S_BSY, S_CD, S_IO, S_MSG, S_REQ, S_RST, S_SEL
- wire segments 538 -> 363
- no-connect marks 14 -> 37
Other:
- note added: "3V"
- note added: "GPIO 0"
- note added: "GPIO 1"
- note added: "←1mA"
- moved on the sheet: D1, F1, R1
