File: scsiemu.sch (KiCad schematic (older format))
At the start: 32 parts, among them J1 RasPi, J2 SCSI, J3 USB_POWER, J4 POWER 5V, J5 I2C, U1 74LS641-1, U2 74LS641-1, U3 74LS641-1, U4 74LS641-1

Commit message: update libs update PCBs update schematic
Parts:
- removed J2: SCSI, local_lib:DSUB50P, symbol local_lib:DSUB_SCSI
- removed J5: I2C, Connector_JST:JST_PH_S3B-PH-K_1x03_P2.00mm_Horizontal, symbol Connector:Conn_01x03_Male
- removed RN10, RN5, RN7, RN8: 220, Resistor_SMD:R_Cat16-8, symbol Device:R_Pack08
- removed RN11, RN6, RN9: 330, Resistor_SMD:R_Cat16-8, symbol Device:R_Pack08
- added C10, C11, C6, C8: 10u, Capacitor_SMD:C_1206_3216Metric_Pad1.42x1.75mm_HandSolder, symbol Device:C
- added C7, C9: 2.2u, Capacitor_SMD:C_0603_1608Metric_Pad1.05x0.95mm_HandSolder, symbol Device:C
- added D2: SBD, local_lib:D_SOD-123_HandSoldering, symbol Device:D_ALT
- added J2: SCSI, Connector_PinHeader_2.54mm:PinHeader_2x25_P2.54mm_Horizontal, symbol Connector_Generic:Conn_02x25_Odd_Even
- added J5: POWER 5V, Connector_JST:JST_XH_B2B-XH-A_1x02_P2.50mm_Vertical, symbol Connector:Conn_01x02_Male
- added J6: AT Power 5V (171826-4), local_lib:Molex_171826-4, symbol Connector_Generic:Conn_01x04
- added J7: I2C Ext, Connector_JST:JST_XH_B6B-XH-A_1x06_P2.50mm_Vertical, symbol Connector_Generic:Conn_01x06
- added J8: AT Power 5V (641737-1), local_lib:TE_641737-1, symbol Connector_Generic:Conn_01x04
- added LED2: LED ACT, LED_SMD:LED_0603_1608Metric_Pad1.05x0.95mm_HandSolder, symbol Device:LED
- added MH1, MH10, MH2, MH3, MH4, MH9: Raspi Mount, MountingHole:MountingHole_2.2mm_M2, symbol Connector_Generic:Conn_01x01
- added MH5, MH6, MH7, MH8: HDD Mount, MountingHole:MountingHole_3.5mm, symbol Connector_Generic:Conn_01x01
- added R2: 2.2k, Resistor_SMD:R_0603_1608Metric_Pad1.05x0.95mm_HandSolder, symbol Device:R
- added R3: 2.7k, Resistor_SMD:R_0603_1608Metric_Pad1.05x0.95mm_HandSolder, symbol Device:R
- added U5, U6: DS2105Z, Package_SO:SOIC-16_3.9x9.9mm_P1.27mm, symbol local_lib:DS2105Z
- added U7, U8: TL2218-285, Package_SO:TSSOP-20_4.4x6.5mm_P0.65mm, symbol local_lib:TL2218-285
- C1, C2, C4: value 0.1u JB -> 0.1u
- C3: value 0.1u JIS B -> 0.1u
- C5: value 10u JB -> 10u
- D1: footprint cd_device:D_SOD-123_HandSoldering -> local_lib:D_SOD-123_HandSoldering
- F2: value 1A -> 2A
- J4: footprint Connector_JST:JST_PH_S2B-PH-K_1x02_P2.00mm_Horizontal -> Connector_JST:JST_XH_B2B-XH-A_1x02_P2.50mm_Vertical
Connections:
- net labels added: 5V_DC, AT_5V_DC, AT_POWER_ON, EXT1, EXT2, S_ACK, S_ATN, S_BSY, S_CD, S_IO, S_MSG, S_REQ, S_RST, S_SEL
- wire segments 538 -> 364
- no-connect marks 14 -> 35
Other:
- note added: "3V"
- note added: "GPIO 0"
- note added: "GPIO 1"
- note added: "←1mA"
- moved on the sheet: D1, F1

Commit message: update track
Parts:
- added R4: 1k, Resistor_SMD:R_0603_1608Metric_Pad1.05x0.95mm_HandSolder, symbol Device:R
- LED1: value LED ACT -> LED PWR; footprint LED_THT:LED_D3.0mm -> LED_SMD:LED_0603_1608Metric_Pad1.05x0.95mm_HandSolder
Connections:
- net 5V_DC: now also LED1.2 (A)
- net ACT: no longer LED1.2 (A)
- net GND: now also R4.2
- net at LED2.1 (K), R1.1: no longer LED1.1 (K)
- new net: LED1.1 (K), R4.1
Other:
- moved on the sheet: LED2, R1
Changed lines of the file:
@@
 	15550 2450 15550 2350
-$Comp
-L Device:LED LED1
-U 1 1 5D2AD275
-P 7300 2850
-F 0 "LED1" V 7338 2732 50  0000 R CNN
-F 1 "LED ACT" V 7247 2732 50  0000 R CNN
-F 2 "LED_THT:LED_D3.0mm" H 7300 2850 50  0001 C CNN
-F 3 "~" H 7300 2850 50  0001 C CNN
-	1    7300 2850
-	0    -1   -1   0
-$EndComp
-Text Label 7300 2600 2    50   ~ 0
-ACT
 $Comp
 L power:VEE #PWR01
@@
 L Device:R R1
 U 1 1 5D381E27
-P 7300 3250
-F 0 "R1" H 7370 3296 50  0000 L CNN
-F 1 "1k" H 7370 3205 50  0000 L CNN
-F 2 "Resistor_SMD:R_0603_1608Metric_Pad1.05x0.95mm_HandSolder" V 7230 3250 50  0001 C CNN
-F 3 "~" H 7300 3250 50  0001 C CNN
-	1    7300 3250
-	1    0    0    -1
-$EndComp
-Wire Wire Line
-	7300 3100 7300 3050
+P 7300 2700
+F 0 "R1" H 7370 2746 50  0000 L CNN
+F 1 "1k" H 7370 2655 50  0000 L CNN
+F 2 "Resistor_SMD:R_0603_1608Metric_Pad1.05x0.95mm_HandSolder" V 7230 2700 50  0001 C CNN
+F 3 "~" H 7300 2700 50  0001 C CNN
+	1    7300 2700
+	1    0    0    -1
+$EndComp
 $Comp
 L power:GND #PWR04
 U 1 1 5D48A02F
-P 7300 3500
-F 0 "#PWR04" H 7300 3250 50  0001 C CNN
-F 1 "GND" H 7305 3327 50  0000 C CNN
-F 2 "" H 7300 3500 50  0001 C CNN
-F 3 "" H 7300 3500 50  0001 C CNN
-	1    7300 3500
-	1    0    0    -1
-$EndComp
-Wire Wire Line
-	7300 3500 7300 3400
+P 7300 2950
+F 0 "#PWR04" H 7300 2700 50  0001 C CNN
+F 1 "GND" H 7305 2777 50  0000 C CNN
+F 2 "" H 7300 2950 50  0001 C CNN
+F 3 "" H 7300 2950 50  0001 C CNN
+	1    7300 2950
+	1    0    0    -1
+$EndComp
+Wire Wire Line
+	7300 2950 7300 2850
 Text Label 6000 5200 0    50   ~ 0
 D4
@@
 	6700 2900 6700 3000
 Wire Wire Line
-	6700 3300 6700 4900
+	6700 3300 6700 3500
 $Comp
 L Connector:Conn_01x02_Male J4
@@
 L Device:LED LED2
 U 1 1 60304D76
-P 7950 2850
-F 0 "LED2" V 7988 2732 50  0000 R CNN
-F 1 "LED ACT" V 7897 2732 50  0000 R CNN
-F 2 "LED_SMD:LED_0603_1608Metric_Pad1.05x0.95mm_HandSolder" H 7950 2850 50  0001 C CNN
-F 3 "~" H 7950 2850 50  0001 C CNN
-	1    7950 2850
+P 7300 2300
+F 0 "LED2" V 7338 2182 50  0000 R CNN
+F 1 "LED ACT" V 7247 2182 50  0000 R CNN
+F 2 "LED_SMD:LED_0603_1608Metric_Pad1.05x0.95mm_HandSolder" H 7300 2300 50  0001 C CNN
+F 3 "~" H 7300 2300 50  0001 C CNN
+	1    7300 2300
 	0    -1   -1   0
 $EndComp
 Wire Wire Line
-	7950 2700 7950 2600
-Wire Wire Line
-	7950 2600 7300 2600
-Wire Wire Line
-	7300 2600 7300 2700
-Wire Wire Line
-	7300 3050 7950 3050
-Wire Wire Line
-	7950 3050 7950 3000
-Connection ~ 7300 3050
-Wire Wire Line
-	7300 3050 7300 3000
+	7300 2050 7300 2150
 $Comp
 L Device:Fuse F1
@@
 Wire Wire Line
 	5200 1700 4800 1700
+Text Label 7300 2050 2    50   ~ 0
+ACT
+Wire Wire Line
+	7300 2450 7300 2550
+$Comp
+L Device:R R4
+U 1 1 602D7B0C
+P 6950 4050
+F 0 "R4" H 7020 4096 50  0000 L CNN
+F 1 "1k" H 7020 4005 50  0000 L CNN
+F 2 "Resistor_SMD:R_0603_1608Metric_Pad1.05x0.95mm_HandSolder" V 6880 4050 50  0001 C CNN
+F 3 "~" H 6950 4050 50  0001 C CNN
+	1    6950 4050
+	1    0    0    -1
+$EndComp
+$Comp
+L power:GND #PWR032
+U 1 1 602D7B12
+P 6950 4300
+F 0 "#PWR032" H 6950 4050 50  0001 C CNN
+F 1 "GND" H 6955 4127 50  0000 C CNN
+F 2 "" H 6950 4300 50  0001 C CNN
+F 3 "" H 6950 4300 50  0001 C CNN
+	1    6950 4300
+	1    0    0    -1
+$EndComp
+Wire Wire Line
+	6950 4300 6950 4200
+$Comp
+L Device:LED LED1
+U 1 1 602D7B19
+P 6950 3650
+F 0 "LED1" V 6988 3532 50  0000 R CNN
+F 1 "LED PWR" V 6897 3532 50  0000 R CNN
+F 2 "LED_SMD:LED_0603_1608Metric_Pad1.05x0.95mm_HandSolder" H 6950 3650 50  0001 C CNN
+F 3 "~" H 6950 3650 50  0001 C CNN
+	1    6950 3650
+	0    -1   -1   0
+$EndComp
+Wire Wire Line
+	6950 3800 6950 3900
+Wire Wire Line
+	6950 3500 6700 3500
+Connection ~ 6700 3500
+Wire Wire Line
+	6700 3500 6700 4900
 $EndSCHEMATC

Commit message: add tracks more
Connections:
- net S_D0: now also U6.11 (R6), U8.17 (D8)
- net S_D1: now also U6.6 (R5), U8.16 (D7)
- net S_D2: now also U6.12 (R7), U8.14 (D6)
- net S_D3: now also U6.5 (R4), U8.13 (D5)
- net S_D4: now also U6.13 (R8), U8.8 (D4)
- net S_D5: now also U6.4 (R3), U8.7 (D3)
- net S_D6: now also U6.3 (R2), U8.6 (D2)
- net S_D7: now also U6.14 (R9), U8.5 (D1)
- net S_DP: now also U6.2 (R1), U8.4 (D0)
Other:
- moved on the sheet: C8, C9, U6
Changed lines of the file:
@@
 L local_lib:DS2105Z U6
 U 1 1 5FB79863
-P 13350 7000
-F 0 "U6" H 13350 8165 50  0000 C CNN
-F 1 "DS2105Z" H 13350 8074 50  0000 C CNN
-F 2 "Package_SO:SOIC-16_3.9x9.9mm_P1.27mm" H 13350 7000 50  0001 C CNN
-F 3 "" H 13350 7000 50  0001 C CNN
-	1    13350 7000
+P 13500 7000
+F 0 "U6" H 13500 8165 50  0000 C CNN
+F 1 "DS2105Z" H 13500 8074 50  0000 C CNN
+F 2 "Package_SO:SOIC-16_3.9x9.9mm_P1.27mm" H 13500 7000 50  0001 C CNN
+F 3 "" H 13500 7000 50  0001 C CNN
+	1    13500 7000
 	-1   0    0    -1
 $EndComp
-NoConn ~ 13900 6750
+NoConn ~ 14050 6750
 $Comp
 L Device:C C9
 U 1 1 5FB7986A
-P 14150 6600
-F 0 "C9" H 14265 6646 50  0000 L CNN
-F 1 "2.2u" H 14265 6555 50  0000 L CNN
-F 2 "Capacitor_SMD:C_0603_1608Metric_Pad1.05x0.95mm_HandSolder" H 14188 6450 50  0001 C CNN
-F 3 "~" H 14150 6600 50  0001 C CNN
-	1    14150 6600
+P 14300 6600
+F 0 "C9" H 14415 6646 50  0000 L CNN
+F 1 "2.2u" H 14415 6555 50  0000 L CNN
+F 2 "Capacitor_SMD:C_0603_1608Metric_Pad1.05x0.95mm_HandSolder" H 14338 6450 50  0001 C CNN
+F 3 "~" H 14300 6600 50  0001 C CNN
+	1    14300 6600
 	1    0    0    -1
 $EndComp
@@
 L Device:C C8
 U 1 1 5FB79870
-P 14450 6300
-F 0 "C8" H 14565 6346 50  0000 L CNN
-F 1 "10u" H 14565 6255 50  0000 L CNN
-F 2 "Capacitor_SMD:C_1206_3216Metric_Pad1.42x1.75mm_HandSolder" H 14488 6150 50  0001 C CNN
-F 3 "~" H 14450 6300 50  0001 C CNN
-	1    14450 6300
+P 14600 6300
+F 0 "C8" H 14715 6346 50  0000 L CNN
+F 1 "10u" H 14715 6255 50  0000 L CNN
+F 2 "Capacitor_SMD:C_1206_3216Metric_Pad1.42x1.75mm_HandSolder" H 14638 6150 50  0001 C CNN
+F 3 "~" H 14600 6300 50  0001 C CNN
+	1    14600 6300
 	1    0    0    -1
 $EndComp
@@
 L power:VCC #PWR018
 U 1 1 5FB79876
-P 14450 6000
-F 0 "#PWR018" H 14450 5850 50  0001 C CNN
-F 1 "VCC" H 14467 6173 50  0000 C CNN
-F 2 "" H 14450 6000 50  0001 C CNN
-F 3 "" H 14450 6000 50  0001 C CNN
-	1    14450 6000
+P 14600 6000
+F 0 "#PWR018" H 14600 5850 50  0001 C CNN
+F 1 "VCC" H 14617 6173 50  0000 C CNN
+F 2 "" H 14600 6000 50  0001 C CNN
+F 3 "" H 14600 6000 50  0001 C CNN
+	1    14600 6000
 	-1   0    0    -1
 $EndComp
 Wire Wire Line
-	13900 6100 14000 6100
-Wire Wire Line
-	14450 6100 14450 6150
-Wire Wire Line
-	14450 6100 14450 6000
-Connection ~ 14450 6100
-Wire Wire Line
-	13900 6200 14000 6200
-Wire Wire Line
-	14000 6200 14000 6100
-Connection ~ 14000 6100
-Wire Wire Line
-	14000 6100 14450 6100
-Wire Wire Line
-	13900 6450 14150 6450
-Wire Wire Line
-	13900 6350 14150 6350
-Wire Wire Line
-	14150 6350 14150 6450
-Connection ~ 14150 6450
-Wire Wire Line
-	14150 6750 14150 6900
-Wire Wire Line
-	14150 6900 13900 6900
-Connection ~ 14150 6900
-Wire Wire Line
-	14150 6900 14150 7000
+	14050 6100 14150 6100
+Wire Wire Line
+	14600 6100 14600 6150
+Wire Wire Line
+	14600 6100 14600 6000
+Connection ~ 14600 6100
+Wire Wire Line
+	14050 6200 14150 6200
+Wire Wire Line
+	14150 6200 14150 6100
+Connection ~ 14150 6100
+Wire Wire Line
+	14150 6100 14600 6100
+Wire Wire Line
+	14050 6450 14300 6450
+Wire Wire Line
+	14050 6350 14300 6350
+Wire Wire Line
+	14300 6350 14300 6450
+Connection ~ 14300 6450
+Wire Wire Line
+	14300 6750 14300 6900
+Wire Wire Line
+	14300 6900 14050 6900
+Connection ~ 14300 6900
+Wire Wire Line
+	14300 6900 14300 7000
 $Comp
 L power:GND #PWR020
 U 1 1 5FB7988C
-P 14150 7000
-F 0 "#PWR020" H 14150 6750 50  0001 C CNN
-F 1 "GND" H 14155 6827 50  0000 C CNN
-F 2 "" H 14150 7000 50  0001 C CNN
-F 3 "" H 14150 7000 50  0001 C CNN
-	1    14150 7000
+P 14300 7000
+F 0 "#PWR020" H 14300 6750 50  0001 C CNN
+F 1 "GND" H 14305 6827 50  0000 C CNN
+F 2 "" H 14300 7000 50  0001 C CNN
+F 3 "" H 14300 7000 50  0001 C CNN
+	1    14300 7000
 	1    0    0    -1
 $EndComp
@@
 L power:GND #PWR019
 U 1 1 5FB79892
-P 14450 6750
-F 0 "#PWR019" H 14450 6500 50  0001 C CNN
-F 1 "GND" H 14455 6577 50  0000 C CNN
-F 2 "" H 14450 6750 50  0001 C CNN
-F 3 "" H 14450 6750 50  0001 C CNN
-	1    14450 6750
-	1    0    0    -1
-$EndComp
-Wire Wire Line
-	14450 6450 14450 6750
+P 14600 6750
+F 0 "#PWR019" H 14600 6500 50  0001 C CNN
+F 1 "GND" H 14605 6577 50  0000 C CNN
+F 2 "" H 14600 6750 50  0001 C CNN
+F 3 "" H 14600 6750 50  0001 C CNN
+	1    14600 6750
+	1    0    0    -1
+$EndComp
+Wire Wire Line
+	14600 6450 14600 6750
 Wire Wire Line
 	15500 3300 15700 3300
@@
 Wire Wire Line
 	6700 3500 6700 4900
+Text Label 12950 6600 2    50   ~ 0
+S_D0
+Text Label 12950 6500 2    50   ~ 0
+S_D1
+Text Label 12950 6700 2    50   ~ 0
+S_D2
+Text Label 12950 6400 2    50   ~ 0
+S_D3
+Text Label 12950 6800 2    50   ~ 0
+S_D4
+Text Label 12950 6300 2    50   ~ 0
+S_D5
+Text Label 12950 6200 2    50   ~ 0
+S_D6
+Text Label 12950 6900 2    50   ~ 0
+S_D7
+Text Label 12950 6100 2    50   ~ 0
+S_DP
+Text Label 12400 6100 0    50   ~ 0
+S_DP
+Text Label 12400 6200 0    50   ~ 0
+S_D7
+Text Label 12400 6300 0    50   ~ 0
+S_D6
+Text Label 12400 6400 0    50   ~ 0
+S_D5
+Text Label 12400 6600 0    50   ~ 0
+S_D3
+Text Label 12400 6700 0    50   ~ 0
+S_D2
+Text Label 12400 6800 0    50   ~ 0
+S_D1
+Text Label 12400 6900 0    50   ~ 0
+S_D0
+Text Label 12400 6500 0    50   ~ 0
+S_D4
 $EndSCHEMATC

Commit message: update outline
Parts:
- added MH11, MH12: HDD Mount, MountingHole:MountingHole_3.5mm, symbol Connector_Generic:Conn_01x01
Connections:
- no-connect marks 35 -> 37
Changed lines of the file:
@@
 Text Label 12400 6500 0    50   ~ 0
 S_D4
+$Comp
+L Connector_Generic:Conn_01x01 MH11
+U 1 1 5F7E04EB
+P 1850 3450
+F 0 "MH11" V 1722 3530 50  0000 L CNN
+F 1 "HDD Mount" V 1813 3530 50  0000 L CNN
+F 2 "MountingHole:MountingHole_3.5mm" H 1850 3450 50  0001 C CNN
+F 3 "~" H 1850 3450 50  0001 C CNN
+	1    1850 3450
+	0    1    1    0
+$EndComp
+NoConn ~ 1850 3250
+$Comp
+L Connector_Generic:Conn_01x01 MH12
+U 1 1 5F7E04F6
+P 1850 3800
+F 0 "MH12" V 1722 3880 50  0000 L CNN
+F 1 "HDD Mount" V 1813 3880 50  0000 L CNN
+F 2 "MountingHole:MountingHole_3.5mm" H 1850 3800 50  0001 C CNN
+F 3 "~" H 1850 3800 50  0001 C CNN
+	1    1850 3800
+	0    1    1    0
+$EndComp
+NoConn ~ 1850 3600
 $EndSCHEMATC

Commit message: add mounting holes
Parts:
- F1: value 1A -> 750mA ~~ 1A (0ZCJ0075FF2E)
- F2: value 2A -> 2A (0685T2000-01)
Changed lines of the file:
@@
 P 6700 3150
 F 0 "F2" V 6503 3150 50  0000 C CNN
-F 1 "2A" V 6594 3150 50  0000 C CNN
+F 1 "2A (0685T2000-01)" V 6594 3150 50  0000 C CNN
 F 2 "Fuse:Fuse_1206_3216Metric_Pad1.42x1.75mm_HandSolder" V 6630 3150 50  0001 C CNN
 F 3 "~" H 6700 3150 50  0001 C CNN
@@
 P 14950 2450
 F 0 "F1" V 14753 2450 50  0000 C CNN
-F 1 "1A" V 14844 2450 50  0000 C CNN
+F 1 "750mA ~~ 1A (0ZCJ0075FF2E)" V 15100 2550 50  0000 C CNN
 F 2 "Fuse:Fuse_1206_3216Metric_Pad1.42x1.75mm_HandSolder" V 14880 2450 50  0001 C CNN
 F 3 "~" H 14950 2450 50  0001 C CNN

Commit message: termination on/off jumper fix GND plane
Parts:
- added JP1: Internal Terminator, Connector_PinHeader_2.54mm:PinHeader_1x02_P2.54mm_Vertical, symbol Device:Jumper
Connections:
- net GND: now also JP1.1
- net INT_TERM: now reaches U5.16 (~PD)
- net INT_TERM: now also U6.16 (~PD), U7.19 (~DISABLE), U8.19 (~DISABLE), JP1.2
- no-connect marks 37 -> 35
Other:
- note added: "16mm spacer for Raspi"
Changed lines of the file:
@@
 	-1   0    0    -1
 $EndComp
-NoConn ~ 13900 2000
 $Comp
 L Device:C C7
@@
 	-1   0    0    -1
 $EndComp
-NoConn ~ 14050 6750
 $Comp
 L Device:C C9
@@
 Wire Wire Line
 	11050 2150 11050 2200
-NoConn ~ 11150 1900
 $Comp
 L power:VCC #PWR024
@@
 Wire Wire Line
 	11200 6900 11200 6950
-NoConn ~ 11300 6650
 $Comp
 L power:VCC #PWR026
@@
 $EndComp
 NoConn ~ 1850 3600
+Text Label 11150 1900 2    50   ~ 0
+INT_TERM
+Text Label 13900 2000 0    50   ~ 0
+INT_TERM
+Text Label 11300 6650 2    50   ~ 0
+INT_TERM
+Text Label 14050 6750 0    50   ~ 0
+INT_TERM
+Text Label 7550 6650 0    50   ~ 0
+INT_TERM
+$Comp
+L Device:Jumper JP1
+U 1 1 5F734F35
+P 7250 6650
+F 0 "JP1" H 7250 6914 50  0000 C CNN
+F 1 "Internal Terminator" H 7250 6823 50  0000 C CNN
+F 2 "Connector_PinHeader_2.54mm:PinHeader_1x02_P2.54mm_Vertical" H 7250 6650 50  0001 C CNN
+F 3 "~" H 7250 6650 50  0001 C CNN
+	1    7250 6650
+	1    0    0    -1
+$EndComp
+Text Notes 1750 900  0    50   ~ 0
+16mm spacer for Raspi
+$Comp
+L power:GND #PWR0105
+U 1 1 5F73C644
+P 6950 6650
+F 0 "#PWR0105" H 6950 6400 50  0001 C CNN
+F 1 "GND" H 6955 6477 50  0000 C CNN
+F 2 "" H 6950 6650 50  0001 C CNN
+F 3 "" H 6950 6650 50  0001 C CNN
+	1    6950 6650
+	1    0    0    -1
+$EndComp
+NoConn ~ 1850 1950
+NoConn ~ 1850 1600
+$Comp
+L power:PWR_FLAG #FLG0104
+U 1 1 5F79A4A5
+P 6700 1700
+F 0 "#FLG0104" H 6700 1775 50  0001 C CNN
+F 1 "PWR_FLAG" H 6700 1874 50  0000 C CNN
+F 2 "" H 6700 1700 50  0001 C CNN
+F 3 "~" H 6700 1700 50  0001 C CNN
+	1    6700 1700
+	1    0    0    -1
+$EndComp
+Connection ~ 6700 1700
 $EndSCHEMATC

Commit message: minor update
Other:
- note added: "GPIO 9"
Changed lines of the file:
@@
 $EndComp
 Connection ~ 6700 1700
+Text Notes 4450 5900 0    50   ~ 0
+GPIO 9
 $EndSCHEMATC
